Commit message: added world

File: description/robot.urdf.xacro (robot description, xacro)
@@ -2,3 +2,4 @@
 <robot xmlns:xacro="http://www.ros.org/wiki/xacro"  name="robot">
     <xacro:include filename = "robot_core.xacro" />
+    <xacro:include filename = "gazebo_control.xacro" />
 </robot>

File: description/robot_core.xacro (robot description, xacro)
@@ -43,4 +43,7 @@
         </xacro:inertial_box>
     </link>
+    <gazebo reference = "chassis">
+        <material>Gazebo/White</material>
+    </gazebo>
     <!--LEFT WHEEL-->
     <joint name="left_wheel_joint" type="continuous">
@@ -66,4 +69,7 @@
         </xacro:inertial_cylinder>
     </link>
+    <gazebo reference = "left_wheel">
+        <material>Gazebo/Red</material>
+    </gazebo>
     <!--RIGHT WHEEL-->
     <joint name="right_wheel_joint" type="continuous">
@@ -89,4 +95,7 @@
         </xacro:inertial_cylinder>
     </link>
+    <gazebo reference = "right_wheel">
+        <material>Gazebo/Red</material>
+    </gazebo>
     <!--ball-->
     <joint name="caster_ball_joint" type="fixed">
@@ -111,3 +120,8 @@
         </xacro:inertial_sphere>
     </link>
+    <gazebo reference = "caster_ball">
+        <material>Gazebo/Black</material>
+        <mu1 value = "0.001"/>
+        <mu2 value = "0.001"/>
+    </gazebo>
 </robot>
